Commit message: cleaned urdf files

File: kuka_gazebo/urdf/kr70_r2100.urdf.xacro (robot description, xacro)
@@ -4,17 +4,5 @@
   <xacro:include filename="$(find kuka_gazebo)/urdf/kr70_r2100_macro.xacro"/>
   <!-- Read additional arguments  -->
-  <xacro:arg name="use_fake_hardware" default="true"/>
-  <xacro:arg name="roundtrip_time" default="0"/>
-  <xacro:arg name="client_ip" default="0.0.0.0"/>
-  <xacro:arg name="client_port" default="59152"/>
   <xacro:arg name="prefix" default=""/>
-  <xacro:arg name="x" default="0"/>
-  <xacro:arg name="y" default="0"/>
-  <xacro:arg name="z" default="0"/>
-  <xacro:arg name="roll" default="0"/>
-  <xacro:arg name="pitch" default="0"/>
-  <xacro:arg name="yaw" default="0"/>
-  <xacro:kuka_kr70_r2100_robot client_ip="$(arg client_ip)" client_port="$(arg client_port)" prefix="$(arg prefix)" use_fake_hardware="$(arg use_fake_hardware)" roundtrip_time="$(arg roundtrip_time)">
-    <origin xyz="$(arg x) $(arg y) $(arg z)" rpy="$(arg roll) $(arg pitch) $(arg yaw)"/>
-  </xacro:kuka_kr70_r2100_robot>
+  <xacro:kuka_kr70_r2100_robot prefix="$(arg prefix)" />
 </robot>

File: kuka_gazebo/urdf/kr70_r2100_macro.xacro (robot description, xacro)
@@ -2,8 +2,7 @@
 <robot xmlns:xacro="http://wiki.ros.org/xacro">
   <xacro:include filename="$(find kuka_gazebo)/urdf/kr_iontec_ros2_control.xacro"/>
-  <xacro:include filename="$(find kuka_gazebo)/urdf/kr_iontec_transmission.xacro"/>
-  <xacro:macro name="kuka_kr70_r2100_robot" params="client_ip client_port prefix use_fake_hardware roundtrip_time *origin">
+  <xacro:macro name="kuka_kr70_r2100_robot" params="prefix">
     <!-- ros2 control instance -->
-    <xacro:kuka_iontec_ros2_control name="${prefix}kr70_r2100" client_ip="${client_ip}" client_port="${client_port}" prefix="${prefix}" use_fake_hardware="${use_fake_hardware}" roundtrip_time="${roundtrip_time}"/>
+    <xacro:kuka_iontec_ros2_control prefix="${prefix}"/>
     <xacro:arg name="pkg_path" default="$(find kuka_gazebo)"/>
     <link name="world"/>
@@ -143,5 +142,4 @@
       <parent link="world"/>
       <child link="${prefix}base_link"/>
-      <xacro:insert_block name="origin"/>
     </joint>
     <joint name="${prefix}joint_1" type="revolute">

File: kuka_gazebo/urdf/kr_iontec_ros2_control.xacro (robot description, xacro)
@@ -1,5 +1,5 @@
 <?xml version="1.0" encoding="UTF-8"?>
 <robot xmlns:xacro="http://www.ros.org/wiki/xacro">
-  <xacro:macro name="kuka_iontec_ros2_control" params="name client_ip client_port prefix use_fake_hardware roundtrip_time">
+  <xacro:macro name="kuka_iontec_ros2_control" params="prefix">
     <ros2_control name="GazeboSimSystem" type="system">
       <hardware>

Commit message: integrating robotiq gripper

File: kuka_gazebo/urdf/kr70_r2100.urdf.xacro (robot description, xacro)
@@ -5,4 +5,5 @@
   <!-- Read additional arguments  -->
   <xacro:arg name="prefix" default=""/>
-  <xacro:kuka_kr70_r2100_robot prefix="$(arg prefix)" />
+  <xacro:arg name="gripper_name" default=""/>
+  <xacro:kuka_kr70_r2100_robot prefix="$(arg prefix)" gripper_name="$(arg gripper_name)"/>
 </robot>

File: kuka_gazebo/urdf/kr70_r2100_macro.xacro (robot description, xacro)
@@ -2,5 +2,8 @@
 <robot xmlns:xacro="http://wiki.ros.org/xacro">
   <xacro:include filename="$(find kuka_gazebo)/urdf/kr_iontec_ros2_control.xacro"/>
-  <xacro:macro name="kuka_kr70_r2100_robot" params="prefix">
+  <xacro:macro name="kuka_kr70_r2100_robot" params="
+    prefix
+    gripper_name
+  ">
     <!-- ros2 control instance -->
     <xacro:kuka_iontec_ros2_control prefix="${prefix}"/>
@@ -139,4 +142,5 @@
       </visual>
     </link>
+    <!--  Joints  -->
     <joint name="${prefix}world-base_link" type="fixed">
       <parent link="world"/>
@@ -206,4 +210,19 @@
       <parent link="${prefix}link_6"/>
     </joint>
+    <!-- Grippers -->
+    <xacro:unless value="${gripper_name == ''}">
+      <xacro:if value="${gripper_name == 'robotiq_2f_85'}">
+        <xacro:include filename="$(find robotiq_description)/urdf/robotiq_2f_85_macro.urdf.xacro" />
+        <xacro:robotiq_gripper prefix="${prefix}" parent="${prefix}link_6">
+          <origin rpy="0.0 ${pi} 0.0" xyz="0.0 0.0 -0.036" />
+        </xacro:robotiq_gripper>
+      </xacro:if>
+      <xacro:if value="${gripper_name == 'robotiq_2f_140'}">
+        <xacro:include filename="$(find robotiq_description)/urdf/robotiq_2f_140_macro.urdf.xacro" />
+        <xacro:robotiq_gripper prefix="${prefix}" parent="${prefix}link_6">
+          <origin rpy="0.0 ${pi} 0.0" xyz="0.0 0.0 -0.036" />
+        </xacro:robotiq_gripper>
+      </xacro:if>
+    </xacro:unless>
   </xacro:macro>
 </robot>
