Commit message: Adjusted inertia of base_link

File: kuka_gazebo/urdf/kr70_r2100_macro.xacro (robot description, xacro)
@@ -7,17 +7,11 @@
     <xacro:kuka_iontec_ros2_control name="${prefix}kr70_r2100" client_ip="${client_ip}" client_port="${client_port}" prefix="${prefix}" use_fake_hardware="${use_fake_hardware}" roundtrip_time="${roundtrip_time}"/>
     <xacro:arg name="pkg_path" default="$(find kuka_gazebo)"/>
-    <link name="ground">
-      <inertial>
-        <inertia ixx="0.0" ixy="0.0" ixz="0.0" iyy="0.0" iyz="0.0" izz="0.0"/>
-        <mass value="0.001"/>
+    <link name="world"/>
+    <link name="${prefix}base_link">
+      <collision>
+        <geometry>
+          <mesh filename="file://$(arg pkg_path)/meshes/kr70_r2100/collision/base_link.stl"/>
+        </geometry>
         <origin rpy="0.0 0.0 0.0" xyz="0.0 0.0 0.0"/>
-      </inertial>
-    </link>
-    <link name="${prefix}base_link">
-      <collision>
-        <geometry>
-          <mesh filename="file://$(arg pkg_path)/meshes/kr70_r2100/collision/base_link.stl"/>
-        </geometry>
-        <origin rpy="-0.0 0.0 -0.0" xyz="0.0 0.0 0.0"/>
       </collision>
       <visual>
@@ -25,10 +19,9 @@
           <mesh filename="file://$(arg pkg_path)/meshes/kr70_r2100/visual/base_link.dae"/>
         </geometry>
-        <origin rpy="-0.0 0.0 -0.0" xyz="0.0 0.0 0.0"/>
-      </visual>
-      <inertial>
-        <inertia ixx="0.0" ixy="0.0" ixz="0.0" iyy="0.0" iyz="0.0" izz="0.0"/>
-        <mass value="0.001"/>
         <origin rpy="0.0 0.0 0.0" xyz="0.0 0.0 0.0"/>
+      </visual>
+      <inertial>
+        <mass value="2.5205E2"/>
+        <inertia ixx="5.40709339054184" ixy="0.0" ixz="0.0" iyy="7.71982652844139" iyz="0.0" izz="9.08867781161129"/>
       </inertial>
     </link>
@@ -147,6 +140,6 @@
       </visual>
     </link>
-    <joint name="${prefix}ground-base_link" type="fixed">
-      <parent link="ground"/>
+    <joint name="${prefix}world-base_link" type="fixed">
+      <parent link="world"/>
       <child link="${prefix}base_link"/>
       <xacro:insert_block name="origin"/>

Commit message: Added robotiq grippers 2f_85 and 2f_140

File: kuka_gazebo/urdf/kr70_r2100_macro.xacro (robot description, xacro)
@@ -1,5 +1,4 @@
 <?xml version="1.0"?>
 <robot xmlns:xacro="http://wiki.ros.org/xacro">
-  <xacro:include filename="$(find kuka_gazebo)/urdf/kr_iontec_ros2_control.xacro"/>
   <xacro:macro name="kuka_kr70_r2100_robot" params="
     prefix
@@ -7,5 +6,4 @@
   ">
     <!-- ros2 control instance -->
-    <xacro:kuka_iontec_ros2_control prefix="${prefix}"/>
     <xacro:arg name="pkg_path" default="$(find kuka_gazebo)"/>
     <link name="world"/>
@@ -211,18 +209,24 @@
     </joint>
     <!-- Grippers -->
-    <xacro:unless value="${gripper_name == ''}">
-      <xacro:if value="${gripper_name == 'robotiq_2f_85'}">
-        <xacro:include filename="$(find robotiq_description)/urdf/robotiq_2f_85_macro.urdf.xacro" />
-        <xacro:robotiq_gripper prefix="${prefix}" parent="${prefix}link_6">
-          <origin rpy="0.0 ${pi} 0.0" xyz="0.0 0.0 -0.036" />
-        </xacro:robotiq_gripper>
-      </xacro:if>
-      <xacro:if value="${gripper_name == 'robotiq_2f_140'}">
-        <xacro:include filename="$(find robotiq_description)/urdf/robotiq_2f_140_macro.urdf.xacro" />
-        <xacro:robotiq_gripper prefix="${prefix}" parent="${prefix}link_6">
-          <origin rpy="0.0 ${pi} 0.0" xyz="0.0 0.0 -0.036" />
-        </xacro:robotiq_gripper>
-      </xacro:if>
-    </xacro:unless>
+    <xacro:if value="${gripper_name != 'robotiq_2f_85' and gripper_name != 'robotiq_2f_140'}">
+        <xacro:include filename="$(find kuka_gazebo)/urdf/kr70_r2100_ros2_control.xacro"/>
+        <xacro:kuka70_r2100_ros2_control prefix="${prefix}"/>
+    </xacro:if>
+    <xacro:if value="${gripper_name == 'robotiq_2f_85'}">
+      <xacro:include filename="$(find kuka_gazebo)/urdf/kr70_r2100_2f85_ros2_control.xacro"/>
+      <xacro:kuka70_r2100_2f85_ros2_control prefix="${prefix}"/>
+      <xacro:include filename="$(find robotiq_description)/urdf/robotiq_2f_85_macro.urdf.xacro" />
+      <xacro:robotiq_gripper prefix="${prefix}" parent="${prefix}link_6">
+        <origin rpy="0.0 ${pi} 0.0" xyz="0.0 0.0 -0.036" />
+      </xacro:robotiq_gripper>
+    </xacro:if>
+    <xacro:if value="${gripper_name == 'robotiq_2f_140'}">
+      <xacro:include filename="$(find kuka_gazebo)/urdf/kr70_r2100_2f140_ros2_control.xacro"/>
+      <xacro:kuka70_r2100_2f140_ros2_control prefix="${prefix}"/>
+      <xacro:include filename="$(find robotiq_description)/urdf/robotiq_2f_140_macro.urdf.xacro" />
+      <xacro:robotiq_gripper prefix="${prefix}" parent="${prefix}link_6">
+        <origin rpy="0.0 ${pi} 0.0" xyz="0.0 0.0 -0.036" />
+      </xacro:robotiq_gripper>
+    </xacro:if>
   </xacro:macro>
 </robot>

File: kuka_gazebo/urdf/kr70_r2100_ros2_control.xacro (robot description, xacro)
@@ -1,5 +1,5 @@
 <?xml version="1.0" encoding="UTF-8"?>
 <robot xmlns:xacro="http://www.ros.org/wiki/xacro">
-  <xacro:macro name="kuka_iontec_ros2_control" params="prefix">
+  <xacro:macro name="kuka70_r2100_ros2_control" params="prefix">
     <ros2_control name="IgnitionSystem" type="system">
       <hardware>
@@ -49,11 +49,11 @@
       </joint>
     </ros2_control>
+    <gazebo>
+        <plugin filename="ign_ros2_control-system" name="ign_ros2_control::IgnitionROS2ControlPlugin">
+            <robot_param>robot_description</robot_param>
+            <robot_param_node>robot_state_publisher</robot_param_node>
+            <parameters>$(find kuka_gazebo)/config/kuka_controllers.yaml</parameters>
+        </plugin>
+    </gazebo>
   </xacro:macro>
-  <gazebo>
-      <plugin filename="ign_ros2_control-system" name="ign_ros2_control::IgnitionROS2ControlPlugin">
-          <robot_param>robot_description</robot_param>
-          <robot_param_node>robot_state_publisher</robot_param_node>
-          <parameters>$(find kuka_gazebo)/config/controllers.yaml</parameters>
-      </plugin>
-  </gazebo>
 </robot>

File: robotiq_description/urdf/2f_85.ros2_control.xacro (robot description, xacro)
@@ -67,9 +67,9 @@
     </xacro:macro>
     <gazebo>
-      <plugin filename="ign_ros2_control-system" name="ign_ros2_control::IgnitionROS2ControlPlugin">
-          <robot_param>robot_description</robot_param>
-          <robot_param_node>robot_state_publisher</robot_param_node>
-          <parameters>$(find robotiq_description)/config/robotiq_controllers.yaml</parameters>
-      </plugin>
-  </gazebo>
+        <plugin filename="ign_ros2_control-system" name="ign_ros2_control::IgnitionROS2ControlPlugin">
+            <robot_param>robot_description</robot_param>
+            <robot_param_node>robot_state_publisher</robot_param_node>
+            <parameters>$(find robotiq_description)/config/robotiq_2f85_controllers.yaml</parameters>
+        </plugin>
+    </gazebo>
 </robot>

File: robotiq_description/urdf/robotiq_2f_140.xacro (robot description, xacro)
@@ -17,5 +17,5 @@
         <origin xyz="0 0 0" rpy="0 0 0" />
         <geometry>
-          <mesh filename="package://robotiq_description/meshes/visual/2f_140/robotiq_2f_${stroke}_outer_knuckle.stl" />
+          <mesh filename="file://$(find robotiq_description)/meshes/visual/2f_140/robotiq_2f_${stroke}_outer_knuckle.stl" />
         </geometry>
         <material name="">
@@ -26,5 +26,5 @@
         <origin xyz="0 0 0" rpy="0 0 0" />
         <geometry>
-          <mesh filename="package://robotiq_description/meshes/collision/2f_140/robotiq_2f_${stroke}_outer_knuckle.stl" />
+          <mesh filename="file://$(find robotiq_description)/meshes/collision/2f_140/robotiq_2f_${stroke}_outer_knuckle.stl" />
         </geometry>
       </collision>
@@ -47,5 +47,5 @@
         <origin xyz="0 0 0" rpy="0 0 0" />
         <geometry>
-          <mesh filename="package://robotiq_description/meshes/visual/2f_140/robotiq_2f_${stroke}_outer_finger.stl" />
+          <mesh filename="file://$(find robotiq_description)/meshes/visual/2f_140/robotiq_2f_${stroke}_outer_finger.stl" />
         </geometry>
         <material name="">
@@ -56,5 +56,5 @@
         <origin xyz="0 0 0" rpy="0 0 0" />
         <geometry>
-          <mesh filename="package://robotiq_description/meshes/collision/2f_140/robotiq_2f_${stroke}_outer_finger.stl" />
+          <mesh filename="file://$(find robotiq_description)/meshes/collision/2f_140/robotiq_2f_${stroke}_outer_finger.stl" />
         </geometry>
       </collision>
@@ -77,5 +77,5 @@
         <origin xyz="0 0 0" rpy="0 0 0" />
         <geometry>
-          <mesh filename="package://robotiq_description/meshes/visual/2f_140/robotiq_2f_${stroke}_inner_knuckle.stl" />
+          <mesh filename="file://$(find robotiq_description)/meshes/visual/2f_140/robotiq_2f_${stroke}_inner_knuckle.stl" />
         </geometry>
         <material name="">
@@ -86,5 +86,5 @@
         <origin xyz="0 0 0" rpy="0 0 0" />
         <geometry>
-          <mesh filename="package://robotiq_description/meshes/collision/2f_140/robotiq_2f_${stroke}_inner_knuckle.stl" />
+          <mesh filename="file://$(find robotiq_description)/meshes/collision/2f_140/robotiq_2f_${stroke}_inner_knuckle.stl" />
         </geometry>
       </collision>
@@ -107,5 +107,5 @@
         <origin xyz="0 0 0" rpy="0 0 0" />
         <geometry>
-          <mesh filename="package://robotiq_description/meshes/visual/2f_140/robotiq_2f_${stroke}_inner_finger.stl" />
+          <mesh filename="file://$(find robotiq_description)/meshes/visual/2f_140/robotiq_2f_${stroke}_inner_finger.stl" />
         </geometry>
         <material name="">
@@ -116,5 +116,5 @@
         <origin xyz="0 0 0" rpy="0 0 0" />
         <geometry>
-          <mesh filename="package://robotiq_description/meshes/collision/2f_140/robotiq_2f_${stroke}_inner_finger.stl" />
+          <mesh filename="file://$(find robotiq_description)/meshes/collision/2f_140/robotiq_2f_${stroke}_inner_finger.stl" />
         </geometry>
       </collision>

File: robotiq_description/urdf/robotiq_2f_140_macro.urdf.xacro (robot description, xacro)
@@ -6,7 +6,7 @@
         *origin">
         <!-- ros2 control include -->
-        <xacro:include filename="$(find robotiq_description)/urdf/2f_140.ros2_control.xacro" />
+        <!-- <xacro:include filename="$(find robotiq_description)/urdf/2f_140.ros2_control.xacro" /> -->
         <!-- if we are simulating or directly communicating with the gripper we need a ros2 control instance -->
-        <xacro:robotiq_gripper_ros2_control prefix="${prefix}"/>
+        <!-- <xacro:robotiq_gripper_ros2_control prefix="${prefix}"/> -->
         <!-- this is a temporary link to rotate the 2f-140 gripper to match the 2f-85 -->
         <link name="${prefix}robotiq_base_link"/>
@@ -25,5 +25,5 @@
           <origin xyz="0 0 0" rpy="0 0 0" />
           <geometry>
-            <mesh filename="package://robotiq_description/meshes/visual/2f_140/robotiq_2f_140_base_link.stl" />
+            <mesh filename="file://$(find robotiq_description)/meshes/visual/2f_140/robotiq_2f_140_base_link.stl" />
           </geometry>
           <material name="">
@@ -34,5 +34,5 @@
           <origin xyz="0 0 0" rpy="0 0 0" />
           <geometry>
-            <mesh filename="package://robotiq_description/meshes/collision/2f_140/robotiq_2f_140_base_link.stl" />
+            <mesh filename="file://$(find robotiq_description)/meshes/collision/2f_140/robotiq_2f_140_base_link.stl" />
           </geometry>
         </collision>

File: robotiq_description/urdf/robotiq_2f_85_macro.urdf.xacro (robot description, xacro)
@@ -6,16 +6,16 @@
         *origin">
         <!-- ros2 control include -->
-        <xacro:include filename="$(find robotiq_description)/urdf/2f_85.ros2_control.xacro" />
+        <!-- <xacro:include filename="$(find robotiq_description)/urdf/2f_85.ros2_control.xacro" /> -->
         <!-- if we are simulating or directly communicating with the gripper we need a ros2 control instance -->
-        <xacro:robotiq_gripper_ros2_control prefix="${prefix}"/>
+        <!-- <xacro:robotiq_gripper_ros2_control prefix="${prefix}"/> -->
         <link name="${prefix}robotiq_85_base_link">
             <visual>
                 <geometry>
-                    <mesh filename="package://robotiq_description/meshes/visual/2f_85/robotiq_base.dae" />
-                </geometry>
-            </visual>
-            <collision>
-                <geometry>
-                    <mesh filename="package://robotiq_description/meshes/collision/2f_85/robotiq_base.stl" />
+                    <mesh filename="file://$(find robotiq_description)/meshes/visual/2f_85/robotiq_base.dae" />
+                </geometry>
+            </visual>
+            <collision>
+                <geometry>
+                    <mesh filename="file://$(find robotiq_description)/meshes/collision/2f_85/robotiq_base.stl" />
                 </geometry>
             </collision>
@@ -29,10 +29,10 @@
             <visual>
                 <geometry>
-                    <mesh filename="package://robotiq_description/meshes/visual/2f_85/left_knuckle.dae" />
-                </geometry>
-            </visual>
-            <collision>
-                <geometry>
-                    <mesh filename="package://robotiq_description/meshes/collision/2f_85/left_knuckle.stl" />
+                    <mesh filename="file://$(find robotiq_description)/meshes/visual/2f_85/left_knuckle.dae" />
+                </geometry>
+            </visual>
+            <collision>
+                <geometry>
+                    <mesh filename="file://$(find robotiq_description)/meshes/collision/2f_85/left_knuckle.stl" />
                 </geometry>
             </collision>
@@ -46,10 +46,10 @@
             <visual>
                 <geometry>
-                    <mesh filename="package://robotiq_description/meshes/visual/2f_85/right_knuckle.dae" />
-                </geometry>
-            </visual>
-            <collision>
-                <geometry>
-                    <mesh filename="package://robotiq_description/meshes/collision/2f_85/right_knuckle.stl" />
+                    <mesh filename="file://$(find robotiq_description)/meshes/visual/2f_85/right_knuckle.dae" />
+                </geometry>
+            </visual>
+            <collision>
+                <geometry>
+                    <mesh filename="file://$(find robotiq_description)/meshes/collision/2f_85/right_knuckle.stl" />
                 </geometry>
             </collision>
@@ -63,10 +63,10 @@
             <visual>
                 <geometry>
-                    <mesh filename="package://robotiq_description/meshes/visual/2f_85/left_finger.dae" />
-                </geometry>
-            </visual>
-            <collision>
-                <geometry>
-                    <mesh filename="package://robotiq_description/meshes/collision/2f_85/left_finger.stl" />
+                    <mesh filename="file://$(find robotiq_description)/meshes/visual/2f_85/left_finger.dae" />
+                </geometry>
+            </visual>
+            <collision>
+                <geometry>
+                    <mesh filename="file://$(find robotiq_description)/meshes/collision/2f_85/left_finger.stl" />
                 </geometry>
             </collision>
@@ -80,10 +80,10 @@
             <visual>
                 <geometry>
-                    <mesh filename="package://robotiq_description/meshes/visual/2f_85/right_finger.dae" />
-                </geometry>
-            </visual>
-            <collision>
-                <geometry>
-                    <mesh filename="package://robotiq_description/meshes/collision/2f_85/right_finger.stl" />
+                    <mesh filename="file://$(find robotiq_description)/meshes/visual/2f_85/right_finger.dae" />
+                </geometry>
+            </visual>
+            <collision>
+                <geometry>
+                    <mesh filename="file://$(find robotiq_description)/meshes/collision/2f_85/right_finger.stl" />
                 </geometry>
             </collision>
@@ -97,10 +97,10 @@
             <visual>
                 <geometry>
-                    <mesh filename="package://robotiq_description/meshes/visual/2f_85/left_inner_knuckle.dae" />
-                </geometry>
-            </visual>
-            <collision>
-                <geometry>
-                    <mesh filename="package://robotiq_description/meshes/collision/2f_85/left_inner_knuckle.stl" />
+                    <mesh filename="file://$(find robotiq_description)/meshes/visual/2f_85/left_inner_knuckle.dae" />
+                </geometry>
+            </visual>
+            <collision>
+                <geometry>
+                    <mesh filename="file://$(find robotiq_description)/meshes/collision/2f_85/left_inner_knuckle.stl" />
                 </geometry>
             </collision>
@@ -114,10 +114,10 @@
             <visual>
                 <geometry>
-                    <mesh filename="package://robotiq_description/meshes/visual/2f_85/right_inner_knuckle.dae" />
-                </geometry>
-            </visual>
-            <collision>
-                <geometry>
-                    <mesh filename="package://robotiq_description/meshes/collision/2f_85/right_inner_knuckle.stl" />
+                    <mesh filename="file://$(find robotiq_description)/meshes/visual/2f_85/right_inner_knuckle.dae" />
+                </geometry>
+            </visual>
+            <collision>
+                <geometry>
+                    <mesh filename="file://$(find robotiq_description)/meshes/collision/2f_85/right_inner_knuckle.stl" />
                 </geometry>
             </collision>
@@ -131,10 +131,10 @@
             <visual>
                 <geometry>
-                    <mesh filename="package://robotiq_description/meshes/visual/2f_85/left_finger_tip.dae" />
-                </geometry>
-            </visual>
-            <collision>
-                <geometry>
-                    <mesh filename="package://robotiq_description/meshes/collision/2f_85/left_finger_tip.stl" />
+                    <mesh filename="file://$(find robotiq_description)/meshes/visual/2f_85/left_finger_tip.dae" />
+                </geometry>
+            </visual>
+            <collision>
+                <geometry>
+                    <mesh filename="file://$(find robotiq_description)/meshes/collision/2f_85/left_finger_tip.stl" />
                 </geometry>
                 <surface>
@@ -166,10 +166,10 @@
             <visual>
                 <geometry>
-                    <mesh filename="package://robotiq_description/meshes/visual/2f_85/right_finger_tip.dae" />
-                </geometry>
-            </visual>
-            <collision>
-                <geometry>
-                    <mesh filename="package://robotiq_description/meshes/collision/2f_85/right_finger_tip.stl" />
+                    <mesh filename="file://$(find robotiq_description)/meshes/visual/2f_85/right_finger_tip.dae" />
+                </geometry>
+            </visual>
+            <collision>
+                <geometry>
+                    <mesh filename="file://$(find robotiq_description)/meshes/collision/2f_85/right_finger_tip.stl" />
                 </geometry>
                 <surface>
