Commit message: Added namespace capability for kuka with robotiq 2f-140 gripper

File: kuka_gazebo/urdf/kr70_r2100_2f140.urdf.xacro (robot description, xacro)
@@ -5,5 +5,16 @@
   <!-- Read additional arguments  -->
   <xacro:arg name="prefix" default=""/>
+  <xacro:arg name="robot_name" default="kuka_arm"/>
+  <xacro:arg name="namespace" default=""/>
   <xacro:arg name="gripper_name" default="robotiq_2f_140"/>
-  <xacro:kuka_kr70_r2100_robot prefix="$(arg prefix)" gripper_name="$(arg gripper_name)"/>
+  <xacro:arg name="controller_file" default="$(find kuka_gazebo)/config/kuka_2f140_controllers.yaml"/>
+  <xacro:kuka_kr70_r2100_robot prefix="$(arg prefix)" robot_name="$(arg robot_name)" gripper_name="$(arg gripper_name)"/>
+  <gazebo>
+    <plugin filename="ign_ros2_control-system" name="ign_ros2_control::IgnitionROS2ControlPlugin">
+        <ros>
+          <namespace>$(arg namespace)</namespace>
+        </ros>
+        <parameters>$(arg controller_file)</parameters>
+    </plugin>
+  </gazebo>
 </robot>

File: kuka_gazebo/urdf/kr70_r2100_2f140_ros2_control.xacro (robot description, xacro)
@@ -1,6 +1,6 @@
 <?xml version="1.0" encoding="UTF-8"?>
 <robot xmlns:xacro="http://www.ros.org/wiki/xacro">
-  <xacro:macro name="kuka70_r2100_2f140_ros2_control" params="prefix">
-    <ros2_control name="IgnitionSystem" type="system">
+  <xacro:macro name="kuka70_r2100_2f140_ros2_control" params="prefix robot_name">
+    <ros2_control name="${robot_name}" type="system">
       <hardware>
           <plugin>ign_ros2_control/IgnitionSystem</plugin>
@@ -77,11 +77,4 @@
       </joint>
     </ros2_control>
-    <gazebo>
-      <plugin filename="ign_ros2_control-system" name="ign_ros2_control::IgnitionROS2ControlPlugin">
-          <robot_param>robot_description</robot_param>
-          <robot_param_node>robot_state_publisher</robot_param_node>
-          <parameters>$(find kuka_gazebo)/config/kuka_2f140_controllers.yaml</parameters>
-      </plugin>
-    </gazebo>
   </xacro:macro>
 </robot>

File: kuka_gazebo/urdf/kr70_r2100_macro.xacro (robot description, xacro)
@@ -3,4 +3,5 @@
   <xacro:macro name="kuka_kr70_r2100_robot" params="
     prefix
+    robot_name
     gripper_name
   ">
@@ -223,5 +224,7 @@
     <xacro:if value="${gripper_name == 'robotiq_2f_140'}">
       <xacro:include filename="$(find kuka_gazebo)/urdf/kr70_r2100_2f140_ros2_control.xacro"/>
-      <xacro:kuka70_r2100_2f140_ros2_control prefix="${prefix}"/>
+      <xacro:kuka70_r2100_2f140_ros2_control
+        prefix="${prefix}"
+        robot_name="${robot_name}"/>
       <xacro:include filename="$(find robotiq_description)/urdf/robotiq_2f_140_macro.urdf.xacro" />
       <xacro:robotiq_gripper prefix="${prefix}" parent="${prefix}link_6">
