Commit message: Added camera to kuka

File: kuka_description/urdf/kr70_r2100_macro.xacro (robot description, xacro)
@@ -7,4 +7,5 @@
   ">
     <!-- ros2 control instance -->
+    <xacro:include filename="$(find kuka_description)/urdf/ign_plugins.xacro" />
     <xacro:arg name="pkg_path" default="$(find kuka_description)"/>
     <link name="world"/>
@@ -141,8 +142,39 @@
       </visual>
     </link>
+    <link name="camera_link">
+      <inertial>
+        <origin xyz="0.011445556188227846 -6.205521900433345e-05 0.019977181929567947" rpy="0 0 0"/>
+        <mass value="0.07410808731596727"/>
+        <inertia ixx="4.8e-05" iyy="7e-06" izz="4.8e-05" ixy="-0.0" iyz="0.0" ixz="0.0"/>
+      </inertial>
+      <visual>
+        <origin xyz="-0.318 0.0 -0.093001" rpy="0 0 0"/>
+        <geometry>
+          <mesh filename="file://$(arg pkg_path)/meshes/kr70_r2100/visual/camera_link.dae" scale="0.001 0.001 0.001"/>
+        </geometry>
+      </visual>
+      <collision>
+        <origin xyz="-0.318 0.0 -0.093001" rpy="0 0 0"/>
+        <geometry>
+          <mesh filename="file://$(arg pkg_path)/meshes/kr70_r2100/visual/camera_link.dae" scale="0.001 0.001 0.001"/>
+        </geometry>
+      </collision>
+    </link>
+    <link name="camera_link_optical"></link>
     <!--  Joints  -->
     <joint name="${prefix}world-base_link" type="fixed">
       <parent link="world"/>
       <child link="${prefix}base_link"/>
+    </joint>
+    <joint name="camera_joint" type="fixed">
+      <child link="camera_link"/>
+      <parent link="${prefix}base_link"/>
+      <origin rpy="0.0 0.5 3.142" xyz="4.0 0.0 3.0"/>
+      <axis xyz="0.0 1.0 0.0"/>
+    </joint>
+        <joint name="camera_optical_joint" type="fixed">
+        <origin xyz="0 0 0" rpy="0 0 0" />
+        <parent link="camera_link" />
+        <child link="camera_link_optical" />
     </joint>
     <joint name="${prefix}joint_1" type="revolute">

Commit message: Modified camera position

File: kuka_description/urdf/kr70_r2100_macro.xacro (robot description, xacro)
@@ -170,5 +170,5 @@
       <child link="camera_link"/>
       <parent link="${prefix}base_link"/>
-      <origin rpy="0.0 0.5 3.142" xyz="4.0 0.0 3.0"/>
+      <origin rpy="0.0 0.5 3.142" xyz="4.5 0.0 3.0"/>
       <axis xyz="0.0 1.0 0.0"/>
     </joint>

Commit message: Modified camera's positioning

File: kuka_description/urdf/kr70_r2100_macro.xacro (robot description, xacro)
@@ -170,5 +170,5 @@
       <child link="camera_link"/>
       <parent link="${prefix}base_link"/>
-      <origin rpy="0.0 0.5 3.142" xyz="4.5 0.0 3.0"/>
+      <origin rpy="0.0 0.5 1.572" xyz="0.0 -4.5 3.0"/>
       <axis xyz="0.0 1.0 0.0"/>
     </joint>
